File: XPE_BLUE/AL8805_XPE_BLUE.kicad_sch (KiCad schematic)
At the start: 17 parts, among them U1 AL8805, U2 C2012X5R1H475K125AB_p, U3 C2012X7R2A104K125AE_p, U4 C3225X7T2J104M160AC_p, U5 TPC_1028_744065330_33u

Commit message: Add files via upload
Correction: XPE blue
Other:
- title: High efficiency 36V/1A buck led driver. XP-E green. -> High efficiency 36V/1A buck led driver. XP-E blue.
Changed lines of the file:
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@@
 	(paper "A4")
 	(title_block
-		(title "High efficiency 36V/1A buck led driver. XP-E green.")
+		(title "High efficiency 36V/1A buck led driver. XP-E blue.")
 		(date "2024-07-11")
 		(rev "1")
